File: PCB/MoovipasShieldESP32/MooviPasShield.kicad_pcb (KiCad board)
At the start: 2 copper layers, 99.1 x 99.9 mm, 15 parts, among them J1 microSD, J2 RFID, J3 BUZZER, J4 LCD_I2C, J5 RTC, J7 PuertosExtra2, J8 VIN, J9 Led, M2 MH2, U1 DoitEsp32Devkit

Commit message: Footprint esp32 modificado
Routing:
- net GND: track 321.7 -> 325.0 mm
- net SDA: track 65.4 -> 62.5 mm
- net +5V: track 181.8 -> 183.8 mm
- net H_CS: track 87.1 -> 85.1 mm
- net RFID_RST: track 109.4 -> 111.1 mm
- net +3V3: track 99.4 -> 100.6 mm
- net V_MOSI: track 42.9 -> 44.1 mm
- net SCL: track 106.1 -> 104.8 mm
- net RST: track 31.3 -> 32.6 mm
- net RFID_CS: track 66.9 -> 68.2 mm
- net H_MOSI: track 46.1 -> 44.8 mm
- net H_MISO: track 48.9 -> 47.6 mm
- net GPIO3: track 10.7 -> 12.0 mm
- net GPIO17: track 22.1 -> 23.4 mm
- net GPIO16: track 21.7 -> 23.0 mm
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
Commit message: Verion de fabricacion
Routing:
- net H_CS: track 85.1 -> 82.7 mm
- net +5V: track 183.8 -> 185.6 mm
- net GND: track 325.0 -> 326.5 mm
- net V_MISO: track 64.0 -> 65.4 mm
